File: Hapsis_PCB/polaris4.1/polaris4.1.kicad_pcb (KiCad board)
At the start: 2 copper layers, 95 x 99 mm, 95 parts, among them J1 Screw_Terminal_01x02, J10 SD CARD, J11 Screw_Terminal_01x02, J12 Screw_Terminal_01x02, J13 Screw_Terminal_01x02, J2 Screw_Terminal_01x02, J3 Screw_Terminal_01x02, J4 Screw_Terminal_01x02, J5 Screw_Terminal_01x02, J6 Screw_Terminal_01x02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

Commit message: updated PCB
Connections:
- A1 pad 8: PYRO_2 -> unconnected-(A1-D5-Pad8)
Changed lines of the file:
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@@
 	(net 69 "Net-(D18-A)")
 	(net 70 "Net-(D19-A)")
+	(net 71 "unconnected-(A1-D5-Pad8)")
 	(footprint "TerminalBlock_Phoenix:TerminalBlock_Phoenix_MKDS-1,5-2_1x02_P5.00mm_Horizontal"
 		(layer "F.Cu")
@@
 			(layers "*.Cu" "*.Mask")
 			(remove_unused_layers no)
-			(net 11 "PYRO_2")
+			(net 71 "unconnected-(A1-D5-Pad8)")
 			(pinfunction "D5")
-			(pintype "bidirectional")
+			(pintype "bidirectional+no_connect")
 			(teardrops
 				(best_length_ratio 0.3)
